Commit message: velocity control

File: src/gazebo_simu/urdf/lds_revolute.urdf.xacro (robot description, xacro)
@@ -13,5 +13,5 @@
     <origin xyz="0 0 0" rpy="0 0 0"/>
     <axis xyz="0 0 1"/>
-    <limit lower="-3.14159" upper="3.14159" effort="100" velocity="0.17453278"/>
+    <limit lower="-0.1" upper="3.14159" effort="100" velocity="0"/>
   </joint>
   <transmission name="lds_revolute_tran">
